File: hardware/proofs_of_concept/Cascaded_74xx165/Cascaded_74xx165.kicad_sch (KiCad schematic)
At the start: 5 parts, among them U501 74LS165, U502 74LS165

Commit message: Added Cascaded 74xx165 breadboard schematic
Other:
- title: Cascaded_74xx165 - Proof of concept -> Cascaded 74xx165 - Proof of concept
Changed lines of the file:
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@@
 	(paper "A5" portrait)
 	(title_block
-		(title "Cascaded_74xx165 - Proof of concept")
+		(title "Cascaded 74xx165 - Proof of concept")
 		(date "2025-08-31")
 		(rev "1.0.&lpha")
@@
 				(at 27.94 162.56 0)
 				(size 12.7 2.54)
-				(margins 0.508 0.508 0 0)
+				(margins 0.508 0.762 0 0)
 				(span 1 1)
 				(fill
@@
 				(at 40.64 162.56 0)
 				(size 93.98 2.54)
-				(margins 0.508 0.508 0 0)
+				(margins 0.508 0.762 0 0)
 				(span 1 1)
 				(fill
@@
 				(at 27.94 165.1 0)
 				(size 12.7 2.54)
-				(margins 0.508 0.508 0 0)
+				(margins 0.508 0.762 0 0)
 				(span 1 1)
 				(fill
@@
 				(at 40.64 165.1 0)
 				(size 93.98 2.54)
-				(margins 0.508 0.508 0 0)
+				(margins 0.508 0.762 0 0)
 				(span 1 1)
 				(fill
@@
 				(at 27.94 167.64 0)
 				(size 12.7 2.54)
-				(margins 0.508 0.508 0 0)
+				(margins 0.508 0.762 0 0)
 				(span 1 1)
 				(fill
@@
 				(at 40.64 167.64 0)
 				(size 93.98 2.54)
-				(margins 0.508 0.508 0 0)
+				(margins 0.508 0.762 0 0)
 				(span 1 1)
 				(fill
@@
 				(at 27.94 170.18 0)
 				(size 12.7 2.54)
-				(margins 0.508 0.508 0 0)
+				(margins 0.508 0.762 0 0)
 				(span 1 1)
 				(fill
@@
 				(at 40.64 170.18 0)
 				(size 93.98 2.54)
-				(margins 0.508 0.508 0 0)
+				(margins 0.508 0.762 0 0)
 				(span 1 1)
 				(fill
@@
 				(at 27.94 172.72 0)
 				(size 12.7 2.54)
-				(margins 0.508 0.508 0 0)
+				(margins 0.508 0.762 0 0)
 				(span 1 1)
 				(fill
@@
 				(at 40.64 172.72 0)
 				(size 93.98 2.54)
-				(margins 0.508 0.508 0 0)
+				(margins 0.508 0.762 0 0)
 				(span 1 1)
 				(fill
@@
 				(at 27.94 175.26 0)
 				(size 12.7 2.54)
-				(margins 0.508 0.508 0 0)
+				(margins 0.508 0.762 0 0)
 				(span 1 1)
 				(fill
@@
 				(at 40.64 175.26 0)
 				(size 93.98 2.54)
-				(margins 0.508 0.508 0 0)
+				(margins 0.508 0.762 0 0)
 				(span 1 1)
 				(fill
@@
 				(at 27.94 177.8 0)
 				(size 12.7 2.54)
-				(margins 0.508 0.508 0 0)
+				(margins 0.508 0.762 0 0)
 				(span 1 1)
 				(fill
@@
 				(at 40.64 177.8 0)
 				(size 93.98 2.54)
-				(margins 0.508 0.508 0 0)
-				(span 1 1)
-				(fill
+				(margins 0.508 0.762 0 0)
+				(span 1 1)
+				(fill
