File: hardware/design/Floating_Signal_Tester.kicad_sch (KiCad schematic)
At the start: 0 parts

Commit message: File cleanup
Added final schematics
Other:
- note added: "Input - Tri-state bus (0V, -12V, floating) Can be pulled up to +6V when there is short circuit on the board under test Output - Digital bus (TTL logic): 5V (true) in case input is floating GND (false) in case output is not floating"
- note removed: "Input - Tri-state bus (0V, -12V, floating) Can be pulled up to +6V when short circuit on board under test Output - Digital bus (TTL logic): 5V (true) in case input is floating GND (false) in case output is not floating"
Changed lines of the file:
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@@
 	(title_block
 		(title "VersaLogic board tester")
-		(date "2025-08-13")
-		(rev "1.0.alpha")
+		(date "2025-09-09")
+		(rev "1.0")
 		(comment 1 "Copyright (c) 2025 by Filip Pynckels & Robin Pynckels")
 	)
-	(text "Input  - Tri-state bus (0V, -12V, floating)\n         Can be pulled up to +6V when short circuit on board under test\n\nOutput - Digital bus (TTL logic): 5V  (true)  in case input is floating\n                                  GND (false) in case output is not floating"
+	(text "Input  - Tri-state bus (0V, -12V, floating)\n         Can be pulled up to +6V when there is short circuit on the board\n         under test\n\nOutput - Digital bus (TTL logic): 5V  (true)  in case input is floating\n                                  GND (false) in case output is not floating"
 		(exclude_from_sim no)
-		(at 29.972 170.434 0)
+		(at 29.972 168.148 0)
 		(effects
 			(font
