File: hardware/design/VersaLogic_Board_Tester.kicad_sch (KiCad schematic)
At the start: 1 part, among them J101 UART

Commit message: File cleanup
Added final schematics
Other:
- note added: "Contains analog signals (+12V to -12V)"
- note added: "Power rails"
- note added: "TTL logic"
Changed lines of the file:
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@@
 	(title_block
 		(title "VersaLogic board tester")
-		(date "2025-08-13")
-		(rev "1.0.alpha")
+		(date "2025-09-09")
+		(rev "1.0")
 		(comment 1 "Copyright (c) 2025 by Filip Pynckels & Robin Pynckels")
+	)
+	(rectangle
+		(start 153.67 111.252)
+		(end 154.94 112.522)
+		(stroke
+			(width 0)
+			(type solid)
+			(color 72 0 0 1)
+		)
+		(fill
+			(type color)
+			(color 255 0 0 0.2509803922)
+		)
+	)
+	(rectangle
+		(start 153.67 113.792)
+		(end 154.94 115.062)
+		(stroke
+			(width 0)
+			(type solid)
+			(color 72 0 0 1)
+		)
+		(fill
+			(type color)
+			(color 0 255 0 0.2509803922)
+		)
+	)
+	(rectangle
+		(start 153.67 116.332)
+		(end 154.94 117.602)
+		(stroke
+			(width 0)
+			(type solid)
+			(color 72 0 0 1)
+		)
+		(fill
+			(type color)
+			(color 255 255 0 0.2509803922)
+		)
+	)
+	(text "Contains analog signals (+12V to -12V)"
+		(exclude_from_sim no)
+		(at 156.21 116.84 0)
+		(effects
+			(font
+				(face "Courier")
+				(size 1.27 1.27)
+				(color 132 0 0 1)
+			)
+			(justify left top)
+		)
+	)
+	(text "TTL logic"
+		(exclude_from_sim no)
+		(at 156.21 114.3 0)
+		(effects
+			(font
+				(face "Courier")
+				(size 1.27 1.27)
+				(color 132 0 0 1)
+			)
+			(justify left top)
+		)
+	)
+	(text "Power rails"
+		(exclude_from_sim no)
+		(at 156.21 111.76 0)
+		(effects
+			(font
+				(face "Courier")
+				(size 1.27 1.27)
+				(color 132 0 0 1)
+			)
+			(justify left top)
+		)
 	)
 	(junction
@@
 		)
 		(fill
-			(color 0 0 0 0.0000)
+			(color 0 255 0 0.2510)
 		)
 		(property "Sheetname" "Direction"
@@
 		)
 		(fill
-			(color 0 0 0 0.0000)
+			(color 0 255 0 0.2510)
 		)
 		(property "Sheetname" "Shift-out Signal"
@@
 		)
 		(fill
-			(color 0 0 0 0.0000)
+			(color 255 255 0 0.2510)
 		)
 		(property "Sheetname" "Board Connector"
@@
 		)
 		(fill
-			(color 0 0 0 0.0000)
+			(color 0 255 0 0.2510)
 		)
 		(property "Sheetname" "Shift-in Floating"
@@
 		)
 		(fill
-			(color 0 0 0 0.0000)
+			(color 0 255 0 0.2510)
 		)
 		(property "Sheetname" "Shift-in Signal"
@@
 		)
 		(fill
-			(color 0 0 0 0.0000)
+			(color 0 255 0 0.2510)
 		)
 		(property "Sheetname" "Controller"
@@
 		)
 		(fill
-			(color 0 0 0 0.0000)
+			(color 255 255 0 0.2510)
 		)
 		(property "Sheetname" "Signal Setter-Getter"
@@
 		)
 		(fill
-			(color 0 0 0 0.0000)
+			(color 255 0 0 0.2510)
 		)
 		(property "Sheetname" "Power Supply"
@@
 		)
 		(fill
-			(color 0 0 0 0.0000)
+			(color 255 255 0 0.2510)
 		)
 		(property "Sheetname" "Floating Signal Tester"
